File: circuit/wombat2/wombat2.kicad_sch (KiCad schematic)
At the start: 120 parts, among them J1 Conn_01x04_Pin, J2 Conn_01x04_Pin, Q1 STD35P6LLF6, Q10 IPB95R130PFD7ATMA1, Q2 STD35P6LLF6, Q9 IPB95R130PFD7ATMA1, U1 2EDN7524FXTMA1, U10 LD1117S33TR_SOT223, U2 L7805, U3 2EDN7524FXTMA1, U4 TMUX1108PW, U5 TSB7191A, U7 ADS1115IDGS, U9 XIAO-ESP32-C3-SMD

Commit message: Update KiCad schematic/PCB; track custom footprint library
- Whitelist Library.pretty/*.kicad_mod in the circuit .gitignore so the
  custom footprints are versioned (symbol libs / fp-lib-table still excluded)
- Update schematic, PCB, and project file

Co-Authored-By: Claude Opus 4.8 (1M context) <noreply@anthropic.com>
Parts:
- removed D3: 1N5819WS, Diode_SMD:D_SMA, symbol Diode:1N5819WS
- added D2, D8: TPSMB600CA-A, Diode_SMD:D_SMA, symbol Diode:SMAJ5.0CA
- added D9: 1N5819WS, Diode_SMD:D_SMA, symbol Diode:1N5819WS
- D1: footprint (none) -> LED_SMD:LED_0805_2012Metric_Pad1.15x1.40mm_HandSolder
- Q10, Q9: value IPB95R130PFD7ATMA1 -> IMBG120R234M2HXTMA1; footprint Package_TO_SOT_SMD:TO-263-2 -> wombat:TO-263-7_TabPin4
- R15, R26, R38, R8: value 3 -> 2.7 ohm
- R41: value 560 -> 270
Connections:
- net +15V: now also F1.2, D9.2 (A); no longer R25.1, R27.1, R28.1
- net COIL_LEFT: now also D2.2 (A2)
- net COIL_RIGHT: now also D8.2 (A2)
- net GND: now also D2.1 (A1), D8.1 (A1)
- new net: D9.1 (K), R25.1, R27.1, R28.1
Other:
- note added: "Gain = 120"
- note removed: "Gain = 59"
- moved on the sheet: C10, C11, C12, C13, C18, C2, C21, C4, C48, C5, C6, C7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

Commit message: Add XIAO-ESP32-C3 footprint with 3D model; update board and schematic
- Add XIAO-ESP32-C3-DIP-SMD footprint to the wombat library (3D model attached)
- Repoint the board's XIAO to the wombat-library footprint
- Update schematic and PCB

Co-Authored-By: Claude Opus 4.8 (1M context) <noreply@anthropic.com>
Parts:
- U9: footprint Seeed Studio XIAO Series Library:XIAO-ESP32-C3-SMD -> wombat:XIAO-ESP32-C3-DIP-SMD
Changed lines of the file:
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@@
 			)
 		)
-		(property "Footprint" "Seeed Studio XIAO Series Library:XIAO-ESP32-C3-SMD"
+		(property "Footprint" "wombat:XIAO-ESP32-C3-DIP-SMD"
 			(at 454.66 107.95 0)
-			(hide yes)
 			(show_name no)
 			(do_not_autoplace no)
